Commit message: 汇总近期导航窄道控制与地图修复
纳入轨迹与航向控制、ROGMap 投影、车体外形、串口接口、现场诊断和修改历史。

File: mas2027_robot_description/urdf/mas2027_sentry.urdf (robot description, URDF)
Before this commit: robot mas2027_sentry, 5 links, 4 joints
Links:
- link base_link: geometry collision box size=0.4271 0.4271 0; visual box size=0.4271 0.4271 0
Joints:
- joint lidar_back_joint: origin xyz=0.00 0.15 0.11 rpy=-0.8389 0 0 -> xyz=0.0176 0.1867 0.1100 rpy=-0.8952 0 0
- joint lidar_joint: origin xyz=0.00 -0.15 0.11 rpy=0.8389 0 0 -> xyz=0.0156 -0.1978 0.1100 rpy=0.8511 0 0
